File: Cyllene.sch (EAGLE design)
At the start: 44 parts, among them IC1 CP2102N-A02-GQFN24, IC4 SCD41-D-R2, J1 SM06B-SRSS-TB, J2 SM02B-SRSS-TB(LF)(SN), Q1 DMG3415U-7, Q2 UMH3NFHATN, SW1 MLL1200S, U1 ESP32-PICO-D4, U4 AP2112K-3.3TRG1

Commit message: Update to documentation
Other:
- note added: "2022-01-26"
- note added: "Battery Charger"
- note added: "Board Holder"
- note added: "ESP32 powered SCD41 based Carbon di Oxide Sensor"
- note added: "Microcontroller"
- note added: "Power"
- note added: "Programming"
- note added: "Sensor"
- note added: "TAN-051-2022-01"
- moved on the sheet: ANT2, C12, C13, C14, C15, C16, C17, C2, C4, C5, D1, IC1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
